File: mcu.kicad_sch (KiCad schematic)
At the start: 32 parts, among them J8 Conn_ARM_SWD_TagConnect_TC203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, J9 Conn_01x05_Pin, SW2 Reset, U1 ${ALTIUM_VALUE}, X1 ${ALTIUM_VALUE}, X2 ${ALTIUM_VALUE}

Commit message: Re-linking the PCB properties back to the schematics
Parts:
- C1, C17, C18, C2: value ${ALTIUM_VALUE} -> 12pF; footprint CAPC1005X04L -> Library:C_0402_1005
- C11: value ${ALTIUM_VALUE} -> 100pF; footprint CAPC1005X04L -> Library:C_0402_1005
- C12, C5, C7, C8: value ${ALTIUM_VALUE} -> 100nF; footprint CAPC1005X04L -> Library:C_0402_1005
- C14, C15: value ${ALTIUM_VALUE} -> 1.0µF; footprint CAPC1608X06L -> Library:C_0603_1608
- C16: value ${ALTIUM_VALUE} -> 47nF; footprint CAPC1005X04L -> Library:C_0402_1005
- C19, C20, C21, C6: value ${ALTIUM_VALUE} -> 4.7µF; footprint CAPC1608X06L -> Library:C_0603_1608
- C3, C4, C9: footprint CAPC1005X04L -> Library:C_0402_1005
- L1: footprint INDC1005X04L -> Library:L_0402_1005
- L2, L4: value ${ALTIUM_VALUE} -> 10µH; footprint INDC1608X06L -> Library:L_0603_1608
- L3: value ${ALTIUM_VALUE} -> 15nH; footprint INDC1005X04L -> Library:L_0402_1005
- LD3: footprint LED_SMD:LED_0201_0603Metric -> Library:LED_0603_1608
- R_BLE1: footprint Resistor_SMD:R_0201_0603Metric -> Library:R_0402_1005
- SW2: footprint Button_Switch_SMD:SW_SPST_B3U-3000P -> Button_Switch_SMD:SW_SPST_B3U-3000P-B
- U1: value ${ALTIUM_VALUE} -> nRF52840-QIAA; footprint AQFN50P700X700X85_HS-74N -> Package_DFN_QFN:Nordic_AQFN-73-1EP_7x7mm_P0.5mm
- X1: value ${ALTIUM_VALUE} -> 32MHz; footprint BT-XTAL_2016 -> NX1612SA-32.000MHZ-CHP:OSCSC105P160X120X35-4N
- X2: value ${ALTIUM_VALUE} -> 32.768kHz; footprint XTAL_3215 -> EXC-1210:XTAL_ECS32761210TR; MANUFACTURER (none) -> *; MANUFACTURER PART NUMBER (none) -> *; PIN COUNT (none) -> 2; PUBLISHER (none) -> Nordic Semiconductor
Changed lines of the file:
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@@
 			)
 		)
-		(property "Value" "${ALTIUM_VALUE}"
+		(property "Value" "10µH"
 			(at 109.22 41.91 0)
 			(effects
@@
 			)
 		)
-		(property "Footprint" "INDC1608X06L"
+		(property "Footprint" "Library:L_0603_1608"
 			(at 115.57 35.56 0)
 			(effects
@@
 			)
 		)
-		(property "Footprint" "Button_Switch_SMD:SW_SPST_B3U-3000P"
+		(property "Footprint" "Button_Switch_SMD:SW_SPST_B3U-3000P-B"
 			(at 229.87 144.78 0)
 			(effects
@@
 			)
 		)
-		(property "Value" "${ALTIUM_VALUE}"
+		(property "Value" "32.768kHz"
 			(at 64.516 67.056 0)
 			(effects
@@
 			)
 		)
-		(property "Footprint" "XTAL_3215"
+		(property "Footprint" "EXC-1210:XTAL_ECS32761210TR"
 			(at 62.23 59.69 0)
 			(effects
@@
 			)
 		)
+		(property "MANUFACTURER" "*"
+			(at 62.23 59.69 0)
+			(effects
+				(font
+					(size 1.27 1.27)
+				)
+				(hide yes)
+			)
+		)
+		(property "MANUFACTURER PART NUMBER" "*"
+			(at 62.23 59.69 0)
+			(effects
+				(font
+					(size 1.27 1.27)
+				)
+				(hide yes)
+			)
+		)
+		(property "PIN COUNT" "2"
+			(at 62.23 59.69 0)
+			(effects
+				(font
+					(size 1.27 1.27)
+				)
+				(hide yes)
+			)
+		)
+		(property "PUBLISHER" "Nordic Semiconductor"
+			(at 62.23 59.69 0)
+			(effects
+				(font
+					(size 1.27 1.27)
+				)
+				(hide yes)
+			)
+		)
 		(pin "1"
 		)
@@
 			)
 		)
-		(property "Value" "${ALTIUM_VALUE}"
+		(property "Value" "100nF"
 			(at 146.812 158.75 0)
 			(effects
@@
 			)
 		)
-		(property "Footprint" "CAPC1005X04L"
+		(property "Footprint" "Library:C_0402_1005"
 			(at 144.78 151.13 0)
 			(effects
@@
 			)
 		)
-		(property "Value" "${ALTIUM_VALUE}"
+		(property "Value" "100pF"
 			(at 205.74 74.422 0)
 			(effects
@@
 			)
 		)
-		(property "Footprint" "CAPC1005X04L"
+		(property "Footprint" "Library:C_0402_1005"
 			(at 203.2 69.85 0)
 			(effects
@@
 			)
 		)
-		(property "Value" "${ALTIUM_VALUE}"
+		(property "Value" "1.0µF"
 			(at 103.886 59.944 0)
 			(effects
@@
 			)
 		)
-		(property "Footprint" "CAPC1608X06L"
+		(property "Footprint" "Library:C_0603_1608"
 			(at 101.6 53.34 0)
 			(effects
@@
 			)
 		)
-		(property "Footprint" "CAPC1005X04L"
+		(property "Footprint" "Library:C_0402_1005"
 			(at 195.58 102.87 0)
 			(effects
@@
 			)
 		)
-		(property "Value" "${ALTIUM_VALUE}"
+		(property "Value" "4.7µF"
 			(at 111.76 149.86 0)
 			(effects
@@
 			)
 		)
-		(property "Footprint" "CAPC1608X06L"
+		(property "Footprint" "Library:C_0603_1608"
 			(at 109.22 142.24 0)
 			(effects
@@
 			)
 		)
-		(property "Value" "${ALTIUM_VALUE}"
+		(property "Value" "47nF"
 			(at 140.97 36.576 0)
 			(effects
@@
 			)
 		)
-		(property "Footprint" "CAPC1005X04L"
+		(property "Footprint" "Library:C_0402_1005"
 			(at 138.43 30.48 0)
 			(effects
@@
 			)
 		)
-		(property "Value" "${ALTIUM_VALUE}"
+		(property "Value" "32MHz"
 			(at 192.786 48.006 0)
 			(effects
@@
 			)
 		)
-		(property "Footprint" "BT-XTAL_2016"
+		(property "Footprint" "NX1612SA-32.000MHZ-CHP:OSCSC105P160X120X35-4N"
 			(at 190.5 48.26 0)
 			(effects
@@
 			)
 		)
-		(property "Footprint" "LED_SMD:LED_0201_0603Metric"
+		(property "Footprint" "Library:LED_0603_1608"
 			(at 248.92 134.62 0)
 			(effects
@@
 			)
 		)
-		(property "Footprint" "CAPC1005X04L"
+		(property "Footprint" "Library:C_0402_1005"
 			(at 213.36 93.98 0)
 			(effects
@@
 			)
 		)
-		(property "Value" "${ALTIUM_VALUE}"
+		(property "Value" "100nF"
 			(at 167.64 60.96 0)
 			(effects
@@
 			)
 		)
-		(property "Footprint" "CAPC1005X04L"
+		(property "Footprint" "Library:C_0402_1005"
 			(at 165.1 53.34 0)
 			(effects
@@
 			)
 		)
-		(property "Value" "${ALTIUM_VALUE}"
+		(property "Value" "100nF"
 			(at 88.9 60.96 0)
 			(effects
@@
 			)
 		)
-		(property "Footprint" "CAPC1005X04L"
+		(property "Footprint" "Library:C_0402_1005"
 			(at 86.36 53.34 0)
 			(effects
@@
 			)
 		)
-		(property "Value" "${ALTIUM_VALUE}"
+		(property "Value" "4.7µF"
 			(at 54.102 129.54 0)
 			(effects
@@
 			)
 		)
-		(property "Footprint" "CAPC1608X06L"
+		(property "Footprint" "Library:C_0603_1608"
 			(at 52.07 121.92 0)
 			(effects
@@
 			)
 		)
-		(property "Footprint" "Resistor_SMD:R_0201_0603Metric"
+		(property "Footprint" "Library:R_0402_1005"
 			(at 248.92 142.24 0)
 			(effects
@@
 			)
 		)
-		(property "Value" "${ALTIUM_VALUE}"
+		(property "Value" "4.7µF"
 			(at 66.04 129.54 0)
 			(effects
@@
 			)
 		)
-		(property "Footprint" "CAPC1608X06L"
+		(property "Footprint" "Library:C_0603_1608"
 			(at 63.5 121.92 0)
 			(effects
@@
 			)
 		)
-		(property "Value" "${ALTIUM_VALUE}"
+		(property "Value" "nRF52840-QIAA"
 			(at 164.338 137.16 0)
 			(effects
@@
 			)
 		)
-		(property "Footprint" "AQFN50P700X700X85_HS-74N"
+		(property "Footprint" "Package_DFN_QFN:Nordic_AQFN-73-1EP_7x7mm_P0.5mm"
 			(at 106.68 132.08 0)
 			(effects
@@
 			)
 		)
-		(property "Value" "${ALTIUM_VALUE}"
+		(property "Value" "12pF"
 			(at 200.66 43.942 0)
 			(effects
@@
 			)
 		)
-		(property "Footprint" "CAPC1005X04L"
+		(property "Footprint" "Library:C_0402_1005"
 			(at 198.12 39.37 0)
 			(effects
@@
 			)
 		)
-		(property "Value" "${ALTIUM_VALUE}"
+		(property "Value" "1.0µF"
 			(at 130.81 36.83 0)
 			(effects
@@
 			)
 		)
-		(property "Footprint" "CAPC1608X06L"
+		(property "Footprint" "Library:C_0603_1608"
 			(at 128.27 38.1 0)
 			(effects
@@
 			)
 		)
-		(property "Value" "${ALTIUM_VALUE}"
+		(property "Value" "15nH"
 			(at 109.22 34.29 0)
 			(effects
@@
 			)
 		)
-		(property "Footprint" "INDC1005X04L"
+		(property "Footprint" "Library:L_0402_1005"
 			(at 115.57 27.94 0)
 			(effects
@@
 			)
 		)
-		(property "Footprint" "INDC1005X04L"
+		(property "Footprint" "Library:L_0402_1005"
 			(at 200.66 86.36 0)
 			(effects
@@
 			)
 		)
-		(property "Value" "${ALTIUM_VALUE}"
+		(property "Value" "100nF"
 			(at 197.612 129.54 0)
 			(effects
@@
 			)
 		)
-		(property "Footprint" "CAPC1005X04L"
+		(property "Footprint" "Library:C_0402_1005"
 			(at 195.58 121.92 0)
 			(effects
@@
 			)
 		)
-		(property "Footprint" "CAPC1005X04L"
+		(property "Footprint" "Library:C_0402_1005"
 			(at 195.58 93.98 0)
 			(effects
@@
 			)
 		)
-		(property "Value" "${ALTIUM_VALUE}"
+		(property "Value" "12pF"
 			(at 200.66 55.372 0)
 			(effects
@@
 			)
 		)
-		(property "Footprint" "CAPC1005X04L"
+		(property "Footprint" "Library:C_0402_1005"
 			(at 198.12 50.8 0)
 			(effects
@@
 			)
 		)
-		(property "Value" "${ALTIUM_VALUE}"
+		(property "Value" "4.7µF"
 			(at 99.06 129.54 0)
 			(effects
@@
 			)
 		)
-		(property "Footprint" "CAPC1608X06L"
+		(property "Footprint" "Library:C_0603_1608"
 			(at 96.52 121.92 0)
 			(effects
@@
 			)
 		)
-		(property "Value" "${ALTIUM_VALUE}"
+		(property "Value" "10µH"
 			(at 90.17 116.84 0)
 			(effects
@@
 			)
 		)
-		(property "Footprint" "INDC1608X06L"
+		(property "Footprint" "Library:L_0603_1608"
 			(at 82.55 116.84 0)
 			(effects
@@
 			)
 		)
-		(property "Value" "${ALTIUM_VALUE}"
+		(property "Value" "12pF"
 			(at 53.34 74.422 0)
 			(effects
@@
 			)
 		)
-		(property "Footprint" "CAPC1005X04L"
+		(property "Footprint" "Library:C_0402_1005"
 			(at 58.42 69.85 0)
 			(effects
@@
 			)
 		)
-		(property "Value" "${ALTIUM_VALUE}"
+		(property "Value" "12pF"
 			(at 53.34 61.722 0)
 			(effects
@@
 			)
 		)
-		(property "Footprint" "CAPC1005X04L"
+		(property "Footprint" "Library:C_0402_1005"
 			(at 58.42 57.15 0)
 			(effects

Commit message: Reworking the PSU block and squeeshing everything into 16x42mm space
Parts:
- C19: value 4.7µF -> 10µF
Connections:
- net Sensor CLK: now also U1.L1 (P0.06)
- net Sensor CS: now also U1.G1 (P0.26)
- net Sensor IRQ: now also U1.N1 (P0.08)
- net Sensor SDIO: now also U1.J1 (P0.04/AIN2)

Commit message: Cleaning up the sensor signals routing
Connections:
- net Sensor CLK: now also U1.A20 (P1.10); no longer U1.L1 (P0.06)
- net Sensor CS: now also U1.A14 (P1.15); no longer U1.G1 (P0.26)
- net Sensor IRQ: now also U1.B19 (P1.11); no longer U1.N1 (P0.08)
- net Sensor SDIO: now also U1.A16 (P1.13); no longer U1.J1 (P0.04/AIN2)
Changed lines of the file:
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@@
 	(symbol
 		(lib_id "npm1100_caax_config1-altium-import:VBUS_BAR")
-		(at 99.06 91.44 270)
+		(at 147.32 60.96 180)
 		(unit 1)
 		(exclude_from_sim no)
@@
 		(dnp no)
 		(property "Reference" "#PWR024"
-			(at 99.06 91.44 0)
+			(at 147.32 60.96 0)
 			(effects
 				(font
@@
 		)
 		(property "Value" "Sensor SDIO"
-			(at 89.916 91.44 90)
+			(at 147.32 51.816 90)
 			(effects
 				(font
@@
 		)
 		(property "Footprint" ""
-			(at 99.06 91.44 0)
+			(at 147.32 60.96 0)
 			(effects
 				(font
@@
 		)
 		(property "Datasheet" ""
-			(at 99.06 91.44 0)
+			(at 147.32 60.96 0)
 			(effects
 				(font
@@
 		)
 		(property "Description" ""
-			(at 99.06 91.44 0)
+			(at 147.32 60.96 0)
 			(effects
 				(font
@@
 	(symbol
 		(lib_id "npm1100_caax_config1-altium-import:VBUS_BAR")
-		(at 99.06 86.36 270)
+		(at 142.24 60.96 180)
 		(unit 1)
 		(exclude_from_sim no)
@@
 		(dnp no)
 		(property "Reference" "#PWR021"
-			(at 99.06 86.36 0)
+			(at 142.24 60.96 0)
 			(effects
 				(font
@@
 		)
 		(property "Value" "Sensor CS"
-			(at 90.678 86.36 90)
+			(at 142.24 52.578 90)
 			(effects
 				(font
@@
 		)
 		(property "Footprint" ""
-			(at 99.06 86.36 0)
+			(at 142.24 60.96 0)
 			(effects
 				(font
@@
 		)
 		(property "Datasheet" ""
-			(at 99.06 86.36 0)
+			(at 142.24 60.96 0)
 			(effects
 				(font
@@
 		)
 		(property "Description" ""
-			(at 99.06 86.36 0)
+			(at 142.24 60.96 0)
 			(effects
 				(font
@@
 	(symbol
 		(lib_id "npm1100_caax_config1-altium-import:VBUS_BAR")
-		(at 99.06 101.6 270)
+		(at 154.94 60.96 180)
 		(unit 1)
 		(exclude_from_sim no)
@@
 		(dnp no)
 		(property "Reference" "#PWR038"
-			(at 99.06 101.6 0)
+			(at 154.94 60.96 0)
 			(effects
 				(font
@@
 		)
 		(property "Value" "Sensor IRQ"
-			(at 90.678 101.6 90)
+			(at 154.94 52.578 90)
 			(effects
 				(font
@@
 		)
 		(property "Footprint" ""
-			(at 99.06 101.6 0)
+			(at 154.94 60.96 0)
 			(effects
 				(font
@@
 		)
 		(property "Datasheet" ""
-			(at 99.06 101.6 0)
+			(at 154.94 60.96 0)
 			(effects
 				(font
@@
 		)
 		(property "Description" ""
-			(at 99.06 101.6 0)
+			(at 154.94 60.96 0)
 			(effects
 				(font
@@
 	(symbol
 		(lib_id "npm1100_caax_config1-altium-import:VBUS_BAR")
-		(at 99.06 96.52 270)
+		(at 157.48 60.96 180)
 		(unit 1)
 		(exclude_from_sim no)
@@
 		(dnp no)
 		(property "Reference" "#PWR037"
-			(at 99.06 96.52 0)
+			(at 157.48 60.96 0)
 			(effects
 				(font
@@
 		)
 		(property "Value" "Sensor CLK"
-			(at 90.678 96.52 90)
+			(at 157.48 52.578 90)
 			(effects
 				(font
@@
 		)
 		(property "Footprint" ""
-			(at 99.06 96.52 0)
+			(at 157.48 60.96 0)
 			(effects
 				(font
@@
 		)
 		(property "Datasheet" ""
-			(at 99.06 96.52 0)
+			(at 157.48 60.96 0)
 			(effects
 				(font
@@
 		)
 		(property "Description" ""
-			(at 99.06 96.52 0)
+			(at 157.48 60.96 0)
 			(effects
 				(font

Commit message: Wiring up the load swiches side of the PCB
Connections:
- net RGB DATA: now also U1.P23 (P1.07)
- net RGB ON: now also U1.A12 (P0.02/AIN0)
- net VSENSE: now also U1.A10 (P0.29/AIN5)
- net VSENSE_ON: now also U1.A8 (P0.31/AIN7)

Commit message: Sorting out most of the powerlines
Connections:
- net LCD CLK: now also U1.AD12 (P0.17)
- net LCD CS: now also U1.AD8 (P0.13)
- net LCD DATA: now also U1.AD10 (P0.15)
- net RGB DATA: now also U1.A12 (P0.02/AIN0); no longer U1.P23 (P1.07)
- net RGB ON: now also U1.P23 (P1.07); no longer U1.A12 (P0.02/AIN0)
Changed lines of the file:
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@@
 	)
 	(symbol
+		(lib_id "npm1100_caax_config1-altium-import:VBUS_BAR")
+		(at 134.62 139.7 0)
+		(unit 1)
+		(exclude_from_sim no)
+		(in_bom yes)
+		(on_board yes)
+		(dnp no)
+		(property "Reference" "#PWR054"
+			(at 134.62 139.7 0)
+			(effects
+				(font
+					(size 1.27 1.27)
+				)
+				(hide yes)
+			)
+		)
+		(property "Value" "LCD CLK"
+			(at 134.62 147.574 90)
+			(effects
+				(font
+					(size 1.27 1.27)
+				)
+			)
+		)
+		(property "Footprint" ""
+			(at 134.62 139.7 0)
+			(effects
+				(font
+					(size 1.27 1.27)
+				)
+			)
+		)
+		(property "Datasheet" ""
+			(at 134.62 139.7 0)
+			(effects
+				(font
+					(size 1.27 1.27)
+				)
+			)
+		)
+		(property "Description" ""
+			(at 134.62 139.7 0)
+			(effects
+				(font
+					(size 1.27 1.27)
+				)
+			)
+		)
+		(pin ""
+		)
+		(instances
+			(project "plan-b"
+				(path "/3a835e6f-a660-4b38-a102-87841cdd95ed/5bb1d2f7-c8fd-447b-99e1-d61ef924696c"
+					(reference "#PWR054")
+					(unit 1)
+				)
+			)
+		)
+	)
+	(symbol
 		(lib_id "power:GND")
 		(at 101.6 60.96 0)
@@
 	(symbol
 		(lib_id "npm1100_caax_config1-altium-import:VBUS_BAR")
-		(at 177.8 99.06 90)
+		(at 137.16 60.96 180)
 		(unit 1)
 		(exclude_from_sim no)
@@
 		(dnp no)
 		(property "Reference" "#PWR049"
-			(at 177.8 99.06 0)
+			(at 137.16 60.96 0)
 			(effects
 				(font
@@
 		)
 		(property "Value" "RGB DATA"
-			(at 186.182 99.06 90)
+			(at 137.16 52.578 90)
 			(effects
 				(font
@@
 		)
 		(property "Footprint" ""
-			(at 177.8 99.06 0)
+			(at 137.16 60.96 0)
 			(effects
 				(font
@@
 		)
 		(property "Datasheet" ""
-			(at 177.8 99.06 0)
+			(at 137.16 60.96 0)
 			(effects
 				(font
@@
 		)
 		(property "Description" ""
-			(at 177.8 99.06 0)
+			(at 137.16 60.96 0)
 			(effects
 				(font
@@
 		)
 		(property "Value" "RST"
-			(at 137.16 143.51 0)
+			(at 137.414 145.542 90)
 			(effects
 				(font
@@
 	)
 	(symbol
+		(lib_id "npm1100_caax_config1-altium-import:VBUS_BAR")
+		(at 124.46 139.7 0)
+		(unit 1)
+		(exclude_from_sim no)
+		(in_bom yes)
+		(on_board yes)
+		(dnp no)
+		(property "Reference" "#PWR056"
+			(at 124.46 139.7 0)
+			(effects
+				(font
+					(size 1.27 1.27)
+				)
+				(hide yes)
+			)
+		)
+		(property "Value" "LCD CS"
+			(at 124.46 148.082 90)
+			(effects
+				(font
+					(size 1.27 1.27)
+				)
+			)
+		)
+		(property "Footprint" ""
+			(at 124.46 139.7 0)
+			(effects
+				(font
+					(size 1.27 1.27)
+				)
+			)
+		)
+		(property "Datasheet" ""
+			(at 124.46 139.7 0)
+			(effects
+				(font
+					(size 1.27 1.27)
+				)
+			)
+		)
+		(property "Description" ""
+			(at 124.46 139.7 0)
+			(effects
+				(font
+					(size 1.27 1.27)
+				)
+			)
+		)
+		(pin ""
+		)
+		(instances
+			(project "plan-b"
+				(path "/3a835e6f-a660-4b38-a102-87841cdd95ed/5bb1d2f7-c8fd-447b-99e1-d61ef924696c"
+					(reference "#PWR056")
+					(unit 1)
+				)
+			)
+		)
+	)
+	(symbol
 		(lib_id "nrf52840_ckaa_var4-altium-import:VDD_nRF_BAR")
 		(at 260.35 52.07 90)
@@
 	)
 	(symbol
+		(lib_id "npm1100_caax_config1-altium-import:VBUS_BAR")
+		(at 129.54 139.7 0)
+		(unit 1)
+		(exclude_from_sim no)
+		(in_bom yes)
+		(on_board yes)
+		(dnp no)
+		(property "Reference" "#PWR055"
+			(at 129.54 139.7 0)
+			(effects
+				(font
+					(size 1.27 1.27)
+				)
+				(hide yes)
+			)
+		)
+		(property "Value" "LCD DATA"
+			(at 129.54 148.082 90)
+			(effects
+				(font
+					(size 1.27 1.27)
+				)
+			)
+		)
+		(property "Footprint" ""
+			(at 129.54 139.7 0)
+			(effects
+				(font
+					(size 1.27 1.27)
+				)
+			)
+		)
+		(property "Datasheet" ""
+			(at 129.54 139.7 0)
+			(effects
+				(font
+					(size 1.27 1.27)
+				)
+			)
+		)
+		(property "Description" ""
+			(at 129.54 139.7 0)
+			(effects
+				(font
+					(size 1.27 1.27)
+				)
+			)
+		)
+		(pin ""
+		)
+		(instances
+			(project "plan-b"
+				(path "/3a835e6f-a660-4b38-a102-87841cdd95ed/5bb1d2f7-c8fd-447b-99e1-d61ef924696c"
+					(reference "#PWR055")
+					(unit 1)
+				)
+			)
+		)
+	)
+	(symbol
 		(lib_id "nrf52840_ckaa_var4-altium-import:VDD_nRF_BAR")
 		(at 177.8 116.84 90)
@@
 	(symbol
 		(lib_id "npm1100_caax_config1-altium-import:VBUS_BAR")
-		(at 137.16 60.96 180)
+		(at 177.8 99.06 90)
 		(unit 1)
 		(exclude_from_sim no)
@@
 		(dnp no)
 		(property "Reference" "#PWR053"
-			(at 137.16 60.96 0)
+			(at 177.8 99.06 0)
 			(effects
 				(font
@@
 		)
 		(property "Value" "RGB ON"
-			(at 137.16 52.578 90)
+			(at 186.182 99.06 90)
 			(effects
 				(font
@@
 		)
 		(property "Footprint" ""
-			(at 137.16 60.96 0)
+			(at 177.8 99.06 0)
 			(effects
 				(font
@@
 		)
 		(property "Datasheet" ""
-			(at 137.16 60.96 0)
+			(at 177.8 99.06 0)
 			(effects
 				(font
@@
 		)
 		(property "Description" ""
-			(at 137.16 60.96 0)
+			(at 177.8 99.06 0)
 			(effects
 				(font
