File: switches.kicad_sch (KiCad schematic)
At the start: 2 parts, among them J4 columns, J6 rows

Commit message: Swapping rows connector to the same 6 pins as columns
Parts:
- J6: symbol Connector:Conn_01x05_Socket -> Connector:Conn_01x06_Socket
Connections:
- new net Row 5: J6.6 (Pin_6)
Changed lines of the file:
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@@
+		)
+	)
+	(hierarchical_label "Row 5"
+		(shape input)
+		(at 102.87 99.06 180)
+		(effects
+			(font
+				(size 1.27 1.27)
+			)
+			(justify right)
 		)
 	)
@@
 	)
 	(symbol
-		(lib_id "Connector:Conn_01x05_Socket")
+		(lib_id "Connector:Conn_01x06_Socket")
 		(at 107.95 91.44 0)
 		(unit 1)
@@
 		(fields_autoplaced yes)
 		(property "Reference" "J6"
-			(at 109.22 90.1699 0)
+			(at 109.22 91.4399 0)
 			(effects
 				(font
@@
 		)
 		(property "Value" "rows"
-			(at 109.22 92.7099 0)
+			(at 109.22 93.9799 0)
 			(effects
 				(font
@@
 			)
 		)
-		(property "Description" "Generic connector, single row, 01x05, script generated"
+		(property "Description" "Generic connector, single row, 01x06, script generated"
 			(at 107.95 91.44 0)
 			(effects
@@
 		(pin "5"
 		)
+		(pin "6"
+		)
 		(instances

Commit message: Optimising for BOM and placements cost reduction
Parts:
- J6: footprint Connector_JST:JST_SH_SM05B-SRSS-TB_1x05-1MP_P1.00mm_Horizontal -> Connector_JST:JST_SH_SM06B-SRSS-TB_1x06-1MP_P1.00mm_Horizontal
Changed lines of the file:
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@@
 			)
 		)
-		(property "Footprint" "Connector_JST:JST_SH_SM05B-SRSS-TB_1x05-1MP_P1.00mm_Horizontal"
+		(property "Footprint" "Connector_JST:JST_SH_SM06B-SRSS-TB_1x06-1MP_P1.00mm_Horizontal"
 			(at 107.95 91.44 0)
 			(effects

Commit message: Further optimising the BOM and adding JLCPCB specific part numbers
Parts:
- J4, J6: LCSC (none) -> C160405
Changed lines of the file:
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@@
+			)
+		)
+		(property "AVAILABILITY" ""
+			(at 107.95 72.39 0)
+			(effects
+				(font
+					(size 1.27 1.27)
+				)
+				(hide yes)
+			)
+		)
+		(property "DESCRIPTION" ""
+			(at 107.95 72.39 0)
+			(effects
+				(font
+					(size 1.27 1.27)
+				)
+				(hide yes)
+			)
+		)
+		(property "PACKAGE" ""
+			(at 107.95 72.39 0)
+			(effects
+				(font
+					(size 1.27 1.27)
+				)
+				(hide yes)
+			)
+		)
+		(property "PRICE" ""
+			(at 107.95 72.39 0)
+			(effects
+				(font
+					(size 1.27 1.27)
+				)
+				(hide yes)
+			)
+		)
+		(property "LCSC" "C160405"
+			(at 107.95 72.39 0)
+			(effects
+				(font
+					(size 1.27 1.27)
+				)
+				(hide yes)
 			)
 		)
@@
 			(at 107.95 91.44 0)
 			(effects
+				(font
+					(size 1.27 1.27)
+				)
+				(hide yes)
+			)
+		)
+		(property "AVAILABILITY" ""
+			(at 107.95 91.44 0)
+			(effects
+				(font
+					(size 1.27 1.27)
+				)
+				(hide yes)
+			)
+		)
+		(property "DESCRIPTION" ""
+			(at 107.95 91.44 0)
+			(effects
+				(font
+					(size 1.27 1.27)
+				)
+				(hide yes)
+			)
+		)
+		(property "PACKAGE" ""
+			(at 107.95 91.44 0)
+			(effects
+				(font
+					(size 1.27 1.27)
+				)
+				(hide yes)
+			)
+		)
+		(property "PRICE" ""
+			(at 107.95 91.44 0)
+			(effects
+				(font
+					(size 1.27 1.27)
+				)
+				(hide yes)
+			)
+		)
+		(property "LCSC" "C160405"
+			(at 107.95 91.44 0)
+			(effects
